File: 74HC597-Breakout.sch (KiCad schematic (older format))
At the start: 17 parts, among them J1 Conn_01x07, J2 Conn_01x07, J3 Conn_01x08, J4 Conn_01x07, J5 Conn_01x07, J6 Conn_01x08, U1 74HC597

Commit message: Local symbols into project lib, also plots
Plotted gerbers and schematic
Moved symbol into a local library
Parts:
- U1: symbol kicad_symbols:74HC597 -> project:74HC597
Changed lines of the file:
@@
 $EndDescr
 $Comp
-L kicad_symbols:74HC597 U1
+L project:74HC597 U1
 U 1 1 5F504068
 P 5300 3400
